File: hardware/hwre.sch (EAGLE design)
At the start: 29 parts

Commit message: updated pcb to hwre v1.1
Parts:
- added 5V, GND: (no value), con-lstb:MA04-1
- added A, B, C, D, E, F, G: (no value), led:LEDCHIP-LED0603
- added C10, C11, C12, C13, C5, C6, C7, C8, C9: (no value), rcl:C-EUC0603
- added EXTRA: (no value), con-lstb:MA10-1
- added TP1, TP2, TP3, TP4, TP5, TP6: TPTP20R, testpad:TPTP20R
- added TP10, TP11, TP12, TP13, TP14, TP15, TP16, TP17, TP18, TP7, TP8, TP9: TPSQTP20R, testpad:TPSQTP20R
- C1, C2, C3, C4: value (none) -> 22pF
- Q1, Q2: value (none) -> 8Mhz
- R1, R2: value (none) -> 2k2
- R10, R11, R6, R7, R8, R9: value (none) -> 68E
- R4, R5: value (none) -> 10K
- renumbered SV1 to BRIDGE, SV2 to LOGIC
Connections:
- removed net 3V3: EEPROM.VCC, PROC1.AVCC, PROC1.VCC@1, PROC2.AVCC, PROC2.VCC@1, R1.2, R2.2, R4.2, R5.2, U$1.CN7_3V3
- new net 5V: 5V.1, 5V.2, 5V.3, 5V.4, EEPROM.VCC, PROC1.AVCC, PROC1.VCC@1, PROC2.AVCC, PROC2.VCC@1, R1.2, R2.2, R4.2, R5.2, U$1.CN7_5V
- new net N$15: PROC1.PB4(MISO), TP2.TP
- new net N$16: PROC1.PB5(SCK), TP3.TP
- new net N$17: PROC2.PB3(MOSI/OC2), TP4.TP
- new net N$18: PROC2.PB4(MISO), TP5.TP
- new net N$19: PROC2.PB5(SCK), TP6.TP
- new net N$20: C7.2, U$1.CN7_25
- new net N$21: C8.2, U$1.CN7_27
- new net N$22: C9.2, U$1.CN7_29
- new net N$23: C10.2, U$1.CN7_31
- new net N$24: C11.2, U$1.CN7_33
- new net N$25: C12.2, U$1.CN7_35
- new net N$26: C13.2, U$1.CN7_37
- new net N$27: C7.1, G.A
- new net N$28: C8.1, F.A
- new net N$29: C9.1, E.A
- new net N$30: C10.1, D.A
- new net N$31: C.A, C11.1
- new net N$32: B.A, C12.1
- new net N$33: A.A, C13.1
- new net N$34: EXTRA.10, U$1.CN10_38
- new net N$35: EXTRA.9, U$1.CN10_36
- new net N$36: EXTRA.8, U$1.CN10_34
- new net N$37: EXTRA.7, U$1.CN10_30
- new net N$38: EXTRA.6, U$1.CN10_28
- new net N$39: EXTRA.5, U$1.CN10_26
- new net N$40: EXTRA.4, U$1.CN10_24
- new net N$41: EXTRA.3, U$1.CN10_22
- new net N$42: EXTRA.2, U$1.CN10_18
- new net N$8: PROC1.PB3(MOSI/OC2), TP1.TP
- new net PC6: C5.2, PROC1.PC6(/RESET), R4.1
- new net PROC2_PC6: C6.2, PROC2.PC6(/RESET), R5.1
- net GND: now also A.C, B.C, C.C, D.C, E.C, EXTRA.1, F.C, G.C, GND.1, GND.2, GND.3, GND.4, TP18.TP
- net PROC1_D1: now also TP17.TP
- net PROC1_D2: now also TP16.TP
- net PROC1_D3: now also TP15.TP
- net PROC1_D4: now also TP14.TP
- net PROC1_D5: now also TP13.TP
- net PROC1_D6: now also TP12.TP
- net PROC1_D7: now also TP11.TP
- net PROC1_D8: now also TP10.TP
- net PROC1_D9: now also TP9.TP
- net PROC1_RESET: now also C5.1; no longer PROC1.PC6(/RESET), R4.1
- net PROC1_SCL: now also TP7.TP
- net PROC1_SDA: now also TP8.TP
- net PROC2_RESET: now also C6.1; no longer PROC2.PC6(/RESET), R5.1
